Commit message: Remove camera, Update colors and modify 'mu' for caster wheel

File: mybot_description/urdf/mybot.xacro (robot description, xacro)
@@ -37,5 +37,5 @@
       <box size="${chassisLength} ${chassisWidth} ${chassisHeight}"/>
     </geometry>
-    <material name="orange"/>
+    <material name="blue"/>
   </visual>
   <inertial>
@@ -76,5 +76,5 @@
 <wheel lr="left" tY="1"/>
 <wheel lr="right" tY="-1"/>
-<joint name="camera_joint" type="continuous">
+<!-- <joint name="camera_joint" type="continuous">
   <parent link="chassis"/>
   <child link="camera"/>
@@ -103,5 +103,5 @@
     <box_inertia m="${cameraMass}" x="${cameraSize}" y="${cameraSize}" z="${cameraSize}" />
   </inertial>
-</link>
+</link> -->
 <joint name="imu_joint" type="continuous">
   <parent link="chassis"/>
